Commit message: config changes

File: src/ros2_com/descriptions/columbus_description.urdf (robot description, URDF)
Before this commit: robot columbus, 4 links, 3 joints
Joints:
- joint lidar_joint: origin xyz=${lidar_xoff} 0 ${lidar_zoff-wheel_radius} rpy=0 0 ${pi} -> xyz=${lidar_xoff} 0 ${lidar_zoff-wheel_radius} rpy=0 0 0
