Commit message: initial point cloud sticher push

File: descriptions/columbus_description.urdf (robot description, URDF)
Before this commit: robot columbus, 4 links, 3 joints
Links:
- added link camera_link; visual box size=0.04 0.12 0.04
Joints:
- added joint camera_joint: type fixed, parent base_link, child camera_link, origin xyz=${lidar_xoff} -0.1 ${lidar_zoff-wheel_radius+0.10} rpy=0 0 0
